File: Electronic/PCB_rigide_test/PCB_rigide.kicad_sch (KiCad schematic)
At the start: 17 parts, among them J1 Conn_01x02_Pin, J2 Conn_01x04_Socket, J3 Conn_01x01_Socket, J4 Conn_01x01_Socket, J5 Conn_01x01_Socket, U2 BMA400, Y1 Crystal_GND24

Commit message: update electronic
Parts:
- added R12, R3, R4, R6, R7, R8, R9: 0, Resistor_SMD:R_1206_3216Metric, symbol Device:R
- AE1: footprint RF_Antenna:Texas_SWRA117D_2.4GHz_Left -> RF_Antenna:Texas_SWRA117D_2.4GHz_Right
- renumbered R4 to R10, R5 to R11, R3 to R5
Connections:
- net GND: now also R6.1, R6.2, R8.1, R8.2, R9.1, R9.2; no longer R2.1, R2.2
- net I2C_SCL: now also R3.1, R3.2
- net I2C_SDA: now also R2.1, R2.2, R4.1, R4.2, R7.1, R7.2
- net RF_TX: now also R12.1, R12.2
- net VCC: now also R10.1, R11.1
- removed net SW0: R10.1, R11.1, U1.6 (SW0)
- no-connect marks 9 -> 10
Other:
- note removed: "SW0 = VCC when IN100 active"
- moved on the sheet: J3, J4, J5, R10, R11
